File: Modellbahn.kicad_sch (KiCad schematic)
At the start: 5 parts, among them J1 CN7, J2 CN10

Commit message: Set doc properties, ignore backups
Other:
- company: (none) -> Jens Böckmann
Changed lines of the file:
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@@
 	(generator_version "8.0")
 	(paper "A4")
+	(title_block
+		(date "2024-12-31")
+		(rev "1")
+		(company "Jens Böckmann")
+	)
 	(junction
 		(at 50.8 45.72)
