File: expansion_a/expansion_a.kicad_pcb (KiCad board)
At the start: 2 copper layers, 60.5 x 56 mm, 47 parts, among them J101 Conn_01x08, J1101 Conn_01x03, J1102 Conn_01x06, J201 Conn_01x03, J202 Conn_01x06, U1001 GAQY212G1S, U101 74HC373, U102 74HC595, U301 GAQY212G1S, U401 GAQY212G1S, U501 GAQY212G1S, U601 GAQY212G1S, U701 GAQY212G1S, U801 GAQY212G1S, U901 GAQY212G1S

Commit message: Error free expansion board
Parts:
- added REF**: MountingHole_3.2mm_M3, MountingHole:MountingHole_3.2mm_M3, F.Cu at (105.9, 62.4)
- added REF**: MountingHole_3.2mm_M3, MountingHole:MountingHole_3.2mm_M3, F.Cu at (147.9, 39.2)
- added REF**: MountingHole_3.2mm_M3, MountingHole:MountingHole_3.2mm_M3, F.Cu at (147.8, 88.1)
- moved J101 24.3 mm to (155.6, 75.5), turned to 90 degrees
- moved J1102 18.0 mm to (107.0, 70.5), turned to -90 degrees
- moved J202 17.5 mm to (107.0, 38.3), turned to -90 degrees
- moved R1001 15.4 mm to (132.1, 88.0)
- moved R301 14.6 mm to (132.9, 39.5)
- moved R901 8.66 mm to (135.4, 88.0)
- moved R401 7.90 mm to (136.1, 39.5)
- moved R701 7.57 mm to (142.0, 88.0)
- moved J1101 6.85 mm to (155.6, 88.3), turned to 90 degrees
- moved J201 6.85 mm to (155.6, 45.3), turned to 90 degrees
- moved R601 5.60 mm to (142.6, 39.5)
- moved R1002 4.23 mm to (117.4, 63.8)
- moved U101 4.08 mm to (116.3, 81.4)
- moved R802 3.57 mm to (117.3, 60.0)
- moved R902 3.56 mm to (120.6, 63.9)
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Connections:
- J101 pad 1: /out1 -> /out8
- J101 pad 2: /out2 -> /out7
- J101 pad 3: /out3 -> /out6
- J101 pad 4: /out4 -> /out5
- J101 pad 5: /out5 -> /out4
- J101 pad 6: /out6 -> /out3
- J101 pad 7: /out7 -> /out2
- J101 pad 8: /out8 -> /out1
Routing:
- net Vdrive: track 0.00 -> 86.3 mm
- net GND: track 0.00 -> 85.1 mm, vias 0 -> 15
- net /set5: track 0.00 -> 80.2 mm
- net VSS: track 0.00 -> 74.9 mm
- net /set6: track 0.00 -> 69.0 mm
- net /set7: track 0.00 -> 67.1 mm
- net /Connector out/CS: track 0.00 -> 62.0 mm, vias 0 -> 1
- net /set4: track 0.00 -> 57.3 mm
- net /Connector in/CS: track 0.00 -> 51.4 mm
- net /set3: track 0.00 -> 47.6 mm
- net /Connector out/CLK: track 0.00 -> 47.0 mm, vias 0 -> 2
- net /set8: track 0.00 -> 46.0 mm
- net GNDPWR: track 0.00 -> 45.7 mm
- net /Connector in/MISO: track 0.00 -> 44.2 mm, vias 0 -> 1
- net /set1: track 0.00 -> 41.5 mm, vias 0 -> 2
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- added copper zone on In1.Cu, net GND
- added copper zone on In2.Cu, net VCC
Other:
- copper layers 2 -> 4

Commit message: Finalise expansion A.
Parts:
- moved J101 41.8 mm to (123.0, 49.3), turned to -90 degrees
- moved REF2 34.2 mm to (113.8, 37.3)
- moved J1101 33.7 mm to (123.0, 79.5), turned to -90 degrees
- moved J201 33.7 mm to (123.0, 36.6), turned to -90 degrees
- moved REF3 33.5 mm to (114.4, 86.4)
- moved R1002 33.4 mm to (84.0, 62.0)
- moved R301 33.4 mm to (99.5, 37.7)
- moved R501 33.4 mm to (105.9, 37.7)
- moved R502 33.4 mm to (84.0, 41.6)
- moved R901 33.4 mm to (102.0, 86.2)
- moved U102 33.4 mm to (85.0, 50.2)
- moved D1001 33.4 mm to (112.6, 81.2)
- moved D301 33.4 mm to (112.6, 42.7)
- moved D401 33.4 mm to (112.6, 48.2)
- moved D501 33.4 mm to (112.6, 53.7)
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- renumbered REF** to REF1, REF** to REF2, REF** to REF3
Connections:
- J101 pad 1: /out8 -> /out1
- J101 pad 2: /out7 -> /out2
- J101 pad 3: /out6 -> /out3
- J101 pad 4: /out5 -> /out4
- J101 pad 5: /out4 -> /out5
- J101 pad 6: /out3 -> /out6
- J101 pad 7: /out2 -> /out7
- J101 pad 8: /out1 -> /out8
Routing:
- net /Connector in/CS: track 51.4 -> 45.5 mm
- net /set5: track 80.2 -> 75.0 mm, vias 0 -> 2
- net /Connector out/CS: track 62.0 -> 59.1 mm
- net /Connector in/CLK: track 28.9 -> 31.8 mm
- net Vdrive: track 86.3 -> 88.7 mm
- net GNDPWR: track 45.7 -> 47.6 mm
- net /set7: track 67.1 -> 65.7 mm
- net /Connector out/MISO: track 7.34 -> 8.53 mm
- net /set6: track 69.0 -> 67.9 mm
- net VSS: track 74.9 -> 75.8 mm
- net Net-(D401-A): track 21.6 -> 20.7 mm
- net /set4: track 57.3 -> 56.4 mm
- net /out5: track 27.0 -> 27.8 mm
- net /out8: track 30.7 -> 31.5 mm
- net /set1: track 41.5 -> 40.7 mm
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Other:
- board size 60.5 x 56 mm -> 58.7 x 55.2 mm
- board text added: "->"
- board text added: "1"
- board text added: "8"
- board text added: "Expansion Board A"
- board text added: "JLCJLCJLCJLC"
- board text added: "Rev: 1"

Commit message: Expander Final II
Parts:
- R1001, R301, R401, R501, R601, R701, R801, R901: value 360 -> 120
- R1002, R302, R402, R502, R602, R702, R802, R902: value 2k4 -> 1k2
- U102: footprint Package_SO:STC_SOP-16_3.9x9.9mm_P1.27mm -> Package_SO:SOIC-16W_5.3x10.2mm_P1.27mm
- moved U102 0.72 mm to (84.3, 50.2)
Routing:
- net Vdrive: track 88.7 -> 0.00 mm
- net VSS: track 75.8 -> 0.00 mm
- net Net-(D801-A): track 22.9 -> 25.9 mm, vias 2 -> 0
- net Net-(JP301-C): track 7.41 -> 10.3 mm
- net /set4: track 56.4 -> 58.9 mm
- net /set1: track 40.7 -> 42.9 mm
- net /set8: track 45.4 -> 47.3 mm
- net /set3: track 46.9 -> 48.6 mm
- net Net-(D701-A): track 28.3 -> 29.2 mm, vias 2 -> 0
- net GND: track 84.6 -> 85.4 mm
- added copper zone on In1.Cu, net VSS
- added copper zone on In2.Cu, net Vdrive
Other:
- board text added: "Modellbahn Expansion Board A"
- board text removed: "Expansion Board A"
