File: expansion_a/output.kicad_sch (KiCad schematic)
At the start: 5 parts, among them U401 GAQY212G1S

Commit message: Finalise expansion A.
Parts:
- JP501: renamed from JP401; now in the parts list
- renumbered D401 to D501, R401 to R501, R402 to R502, U401 to U501
Changed lines of the file:
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@@
 		(unit 1)
 		(exclude_from_sim yes)
-		(in_bom no)
+		(in_bom yes)
 		(on_board yes)
 		(dnp no)
-		(property "Reference" "JP401"
+		(property "Reference" "JP501"
 			(at 133.35 53.34 0)
 			(effects
@@
 		(dnp no)
 		(fields_autoplaced yes)
-		(property "Reference" "R402"
+		(property "Reference" "R502"
 			(at 114.3 63.4999 0)
 			(effects
@@
 		(dnp no)
 		(fields_autoplaced yes)
-		(property "Reference" "D401"
+		(property "Reference" "D501"
 			(at 106.68 73.9774 90)
 			(effects
@@
 		(dnp no)
 		(fields_autoplaced yes)
-		(property "Reference" "R401"
+		(property "Reference" "R501"
 			(at 105.41 60.9599 0)
 			(effects
@@
 		(dnp no)
 		(fields_autoplaced yes)
-		(property "Reference" "U401"
+		(property "Reference" "U501"
 			(at 120.65 69.85 0)
 			(effects

Commit message: Expander Final II
Parts:
- D501: LCSC C5246350 -> C2290
- R501: value 360 -> 120; LCSC C25308 -> C17437
- R502: value 2k4 -> 1k2; LCSC C26018 -> C17379
Connections:
- net set(+5V) renamed set(3V3)
Other:
- company: (none) -> JensBöckmann
- title: (none) -> Output
Changed lines of the file:
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@@
 	(generator_version "8.0")
 	(paper "A4")
+	(title_block
+		(title "Output")
+		(date "2025-01-01")
+		(rev "1")
+		(company "JensBöckmann")
+	)
 	(junction
 		(at 102.87 81.28)
@@
 		)
 	)
-	(text_box "Solid State relais calculation:\nInput Voltage:	5V\nLED Voltage: 	1.2V, 1.4V max\n\nLED operationg Current:			0.6mA,  1.5mA max\nmax. continuous LED current:	50mA\n\nR = (5V-1.4V)/(1.5mA) = 2k4R"
+	(text_box "Solid State relais calculation:\nInput Voltage:			3.3V\nLED Voltage: 			1.2V, 1.4V max\n\nLED operationg Current:	0.6mA,  1.5mA max\nmax. cont. LED current:	50mA\n\nR =	(3.3V-1.4V)/(1.5mA)	= 1k2R"
 		(exclude_from_sim no)
-		(at 88.9 30.48 0)
-		(size 71.12 17.78)
+		(at 95.25 29.21 0)
+		(size 53.34 17.78)
 		(stroke
 			(width 0)
@@
 		)
 	)
+	(text_box "status  calculation:\nInput Voltage:			3.3V\nLED Voltage: 			2.9V\n\nLED operationg Current:	5mA\n\nR = (3.3V-2.9V)/(5mA)	= 120R"
+		(exclude_from_sim no)
+		(at 44.45 57.15 0)
+		(size 39.37 17.78)
+		(stroke
+			(width 0)
+			(type default)
+		)
+		(fill
+			(type none)
+		)
+		(effects
+			(font
+				(size 1.27 1.27)
+			)
+			(justify left top)
+		)
+	)
 	(hierarchical_label "V_drive"
 		(shape passive)
@@
 		)
 	)
-	(hierarchical_label "set(+5V)"
+	(hierarchical_label "set(3V3)"
 		(shape passive)
 		(at 97.79 55.88 180)
@@
 			)
 		)
-		(property "Value" "2k4"
+		(property "Value" "1k2"
 			(at 114.3 66.0399 0)
 			(effects
@@
 			)
 		)
-		(property "LCSC" "C26018"
+		(property "LCSC" "C17379"
 			(at 111.76 64.77 0)
 			(effects
@@
 			)
 		)
-		(property "LCSC" "C5246350"
+		(property "LCSC" "C2290"
 			(at 102.87 73.66 0)
 			(effects
@@
 			)
 		)
-		(property "Value" "360"
+		(property "Value" "120"
 			(at 105.41 63.4999 0)
 			(effects
@@
 			)
 		)
-		(property "LCSC" "C25308"
+		(property "LCSC" "C17437"
 			(at 102.87 62.23 0)
 			(effects
